File: reviung34Mk-II/pcb/bottom-plate-pcb/reviung34-split-BOTTOM.kicad_pcb (KiCad board)
At the start: 2 copper layers, 202.7 x 100 mm, 16 parts

Commit message: Modified to use Kailh hotswaps
Parts:
- removed G***: LOGO, _reviung-kbd:R-x4-ver1
- removed G***: LOGO, _reviung-kbd:REVIUNG34-split-BP-L-logo-ver2
- removed G***: LOGO, _reviung-kbd:REVIUNG34-split-BP-R-logo-ver2
Other:
- board text removed: "REVIUNG34 SPLIT rev 2.0 Designed by gtips 2020"
