File: reviung34Mk-II/pcb/main-pcb/reviung34-split-L.sch (KiCad schematic (older format))
At the start: 74 parts, among them J1 8P8C, J2 8P8C, SW1 SW_PUSH, SW10 SW_PUSH, SW11 SW_PUSH, SW12 SW_PUSH, SW13 SW_PUSH, SW14 SW_PUSH, SW15 SW_PUSH, SW16 SW_PUSH, SW17 SW_PUSH, SW18 SW_PUSH, SW19 SW_PUSH, SW2 SW_PUSH, SW20 SW_PUSH, SW21 SW_PUSH, SW22 SW_PUSH, SW23 SW_PUSH, SW24 SW_PUSH, SW25 SW_PUSH, SW26 SW_PUSH, SW27 SW_PUSH, SW28 SW_PUSH, SW29 SW_PUSH, SW3 SW_PUSH, SW30 SW_PUSH, SW31 SW_PUSH, SW32 SW_PUSH, SW33 SW_PUSH, SW34 SW_PUSH, SW35 SW_PUSH, SW4 SW_PUSH, SW5 SW_PUSH, SW6 SW_PUSH, SW7 SW_PUSH, SW8 SW_PUSH, SW9 SW_PUSH, U1 ProMicro_r

Commit message: Modified to use Kailh hotswaps
Parts:
- J1, J2: symbol _reviung-kbd:8P8C -> reviung34-split-L-rescue:8P8C-_reviung-kbd
- RESET1: symbol _reviung-kbd:SW_PUSH -> reviung34-split-L-rescue:SW_PUSH-_reviung-kbd
- SW1, SW10, SW11, SW12, SW13, SW14, SW15, SW16, SW19, SW2, SW20, SW21, SW22, SW23, SW24, SW25, SW26, SW27, SW28, SW29, SW3, SW30, SW31, SW32, SW33, SW4, SW5, SW6, SW7, SW8, SW9: footprint _reviung-kbd:MXOnly-1U-NoLED -> kbd:CherryMX_Hotswap; symbol _reviung-kbd:SW_PUSH -> reviung34-split-L-rescue:SW_PUSH-_reviung-kbd
- SW17: footprint _reviung-kbd:MXOnly-1U-5pinRcut -> kbd:CherryMX_Hotswap; symbol _reviung-kbd:SW_PUSH -> reviung34-split-L-rescue:SW_PUSH-_reviung-kbd
- SW18: footprint _reviung-kbd:MXOnly-1U-5pinLcut -> kbd:CherryMX_Hotswap; symbol _reviung-kbd:SW_PUSH -> reviung34-split-L-rescue:SW_PUSH-_reviung-kbd
- SW34, SW35: footprint _reviung-kbd:MXOnly-2U-NoLED -> kbd:CherryMX_Hotswap; symbol _reviung-kbd:SW_PUSH -> reviung34-split-L-rescue:SW_PUSH-_reviung-kbd
- U1: symbol _reviung-kbd:ProMicro_r -> reviung34-split-L-rescue:ProMicro_r-_reviung-kbd
