File: reviung34Mk-II/pcb/top-plate-pcb/reviung34-split-L-TOP.kicad_pcb (KiCad board)
At the start: 2 copper layers, 202.7 x 101.5 mm, 21 parts

Commit message: Modified to use Kailh hotswaps
Parts:
- removed G***: LOGO, _reviung-kbd:R-x4-ver1
Other:
- board text removed: "REVIUNG34 SPLIT rev 2.0 Designed by gtips 2020"
